File: PowerSupply.sch (KiCad schematic (older format))
At the start: 15 parts, among them CON1 DC_IN, U1 7805, U5 3.3VREG

Commit message: This branch uses a MCP2200 rather than an FTDI chip
Signed-off-by: Kolijn Wolfaardt <kolijn.wolfaardt@gmail.com>
Parts:
- added C18: 100nF, ~, symbol C
Connections:
- net +5V: now also C18.1
- net GND: now also C18.2
Changed lines of the file:
@@
 LIBS:FT230x
 LIBS:33vReg
+LIBS:mcp2200
 LIBS:Robotics Board-cache
 EELAYER 27 0
@@
 	8400 5300 8400 5400
 Wire Wire Line
-	7850 5950 8650 5950
+	7300 5950 8650 5950
 Wire Wire Line
 	8400 5800 8400 6000
@@
 $EndComp
 Connection ~ 8650 5300
-Text GLabel 7350 5300 0    60   Input ~ 0
+Text GLabel 7000 5300 0    60   Input ~ 0
 Vdd
 Wire Wire Line
-	7350 5300 7500 5300
+	7000 5300 7500 5300
 Text GLabel 8800 5300 2    60   Input ~ 0
 V3.3
@@
 Wire Wire Line
 	7850 5950 7850 5600
+$Comp
+L C C18
+U 1 1 5354577E
+P 7300 5600
+F 0 "C18" H 7300 5700 40  0000 L CNN
+F 1 "100nF" H 7306 5515 40  0000 L CNN
+F 2 "~" H 7338 5450 30  0000 C CNN
+F 3 "~" H 7300 5600 60  0000 C CNN
+	1    7300 5600
+	1    0    0    -1
+$EndComp
+Wire Wire Line
+	7300 5950 7300 5800
+Connection ~ 7850 5950
+Wire Wire Line
+	7300 5400 7300 5300
+Connection ~ 7300 5300
 $EndSCHEMATC
